Commit message: Fix SLAM and navigation by removing rear laser and fixing topic namespacing
- Remove rear laser from URDF - robot now has single front laser only
- Remove rear laser bridge configuration
- Remove laser scan merger from launch file (no longer needed)
- Fix bridge topic namespacing for SLAM and Nav2 compatibility:
  * /scan_raw -> /scan (via scan_frame_relay.py)
  * /odom (was /summit/odom)
  * /cmd_vel (was /summit/cmd_vel)
  * /tf (was /summit/tf)
- Add scan_frame_relay.py to convert Gazebo's scoped frame names
- Update CMakeLists.txt to install scan_frame_relay.py

This fixes SLAM map generation and enables robot navigation.

🤖 Generated with [Claude Code](https://claude.com/claude-code)

Co-Authored-By: Claude <noreply@anthropic.com>

File: icclab_summit_xl/icclab_summit_xl/robots/summit_xls_icclab.urdf.xacro (robot description, xacro)
@@ -33,7 +33,4 @@
 	<xacro:property name="front_laser_offset_y" value="-0.251"/>
 	<xacro:property name="front_laser_offset_z" value="0.1566"/>
-    <xacro:property name="rear_laser_offset_x" value="-0.35"/>
-	<xacro:property name="rear_laser_offset_y" value="0.251"/>
-	<xacro:property name="rear_laser_offset_z" value="0.1566"/>
 	<xacro:property name="front_ptz_camera_offset_x" value="0.308"/>
 	<xacro:property name="front_ptz_camera_offset_y" value="0.141"/>
@@ -86,7 +83,5 @@
 			<origin xyz="${front_laser_offset_x} ${front_laser_offset_y} ${front_laser_offset_z}" rpy="0 0 ${-1/4*PI}" />
   		</xacro:sensor_hokuyo_utm30lx_no_frame_prefix>
-        <xacro:sensor_hokuyo_utm30lx_no_frame_prefix ns="$(arg robot_ns)" prefix="rear_laser" parent="base_link" min_angle="${-3/4*PI}" max_angle="${3/4*PI}" gpu="false">
-			<origin xyz="${rear_laser_offset_x} ${rear_laser_offset_y} ${rear_laser_offset_z}" rpy="0 0 ${3/4*PI}" />
-  		</xacro:sensor_hokuyo_utm30lx_no_frame_prefix>
+		<!-- Rear laser removed - using only front laser -->
 		<!--xacro:sensor_axis_m5013 prefix="$(arg prefix)front_ptz_camera" parent="$(arg prefix)base_link">
 			<origin xyz="${front_ptz_camera_offset_x} ${front_ptz_camera_offset_y} ${front_ptz_camera_offset_z}" rpy="${-PI/2} 0 0"/>
