Commit message: Replace Orbbec Astra with Intel RealSense D435i and remove Luxonis camera
Changes:
- Replaced Orbbec Astra RGBD camera with Intel RealSense D435i for front_rgbd_camera
- Removed Luxonis OAK-D PRO camera (arm_camera)
- Removed unused sensor includes (Orbbec Astra, Luxonis OAK-D PRO)
- Verified camera is publishing data correctly (~4 Hz color, ~6 Hz depth)
- Navigation and SLAM systems confirmed operational

🤖 Generated with [Claude Code](https://claude.com/claude-code)

Co-Authored-By: Claude <noreply@anthropic.com>

File: robots/summit_xl_no_arm.urdf.xacro (robot description, xacro)
@@ -14,9 +14,6 @@
 	<!-- Import our modified sensor -->
 	<xacro:include filename="$(find icclab_summit_xl)/urdf/sensors/hokuyo_utm30lx_no_frame_prefix.urdf.xacro" />
-	<xacro:include filename="$(find icclab_summit_xl)/urdf/sensors/orbbec_astra.urdf.xacro" />
 	<xacro:include filename="$(find icclab_summit_xl)/urdf/sensors/intel_d435.urdf.xacro" />
 	<xacro:include filename="$(find icclab_summit_xl)/urdf/sensors/intel_camera_mount.urdf.xacro" />
-	<xacro:include filename="$(find icclab_summit_xl)/urdf/sensors/luxonis_oak_d_pro.urdf.xacro" />
-	<xacro:include filename="$(find icclab_summit_xl)/urdf/sensors/luxonis_camera_mount.urdf.xacro" />
 	<xacro:include filename="$(find icclab_summit_xl)/urdf/sensors/imu_hector_plugin.urdf.xacro"/>
 	<!-- Arm and gripper removed for no-arm configuration -->
@@ -92,15 +89,11 @@
 			<origin xyz="${rear_ptz_camera_offset_x} ${rear_ptz_camera_offset_y} ${rear_ptz_camera_offset_z}" rpy="${-PI/2} 0 ${PI}"/>
 		</xacro:sensor_axis_m5013-->
-		<xacro:sensor_orbbec_astra_icclab prefix="$(arg prefix)front_rgbd_camera" parent="$(arg prefix)base_link" ns="$(arg robot_ns)">
+		<xacro:sensor_d435_icclab prefix="$(arg prefix)front_rgbd_camera" parent="$(arg prefix)base_link" ns="$(arg robot_ns)">
 			<origin xyz="${front_rgbd_camera_offset_x} ${front_rgbd_camera_offset_y} ${front_rgbd_camera_offset_z}" rpy="0 0 0"/>
-		</xacro:sensor_orbbec_astra_icclab>
+		</xacro:sensor_d435_icclab>
 		<!--xacro:sensor_gps prefix="$(arg prefix)gps" parent="$(arg prefix)base_link">
 			<origin xyz="${gps_offset_x} ${gps_offset_y} ${gps_offset_z}" rpy="0 0 0"/>
 		</xacro:sensor_gps-->
-		<!-- Arm, gripper, and arm camera mount removed -->
-		<!-- Luxonis OAK_D_PRO - repositioned to front chassis from arm -->
-		<xacro:luxonis_oak_icclab prefix="arm_camera" ns="$(arg robot_ns)" parent="$(arg prefix)base_link">
-			   <origin xyz="0.40 0.0 0.25" rpy="0 0 0"/>
-		</xacro:luxonis_oak_icclab>
+		<!-- Arm, gripper, and Luxonis camera removed -->
    </xacro:macro>
    <xacro:summit_xl prefix="$(arg prefix)" publish_bf="true" hq="true"/>

Commit message: Remove rear laser and reposition front laser to center
- Remove rear laser sensor and properties from URDF
- Reposition front laser to center of robot (y: -0.251 -> 0.0)
- Raise front laser height to avoid chassis obstruction (z: 0.1566 -> 0.25)
- Rotate front laser to face forward (rpy: -45° -> 0°)
- Update RViz configuration

This ensures the laser scanning beam is unobstructed by the robot chassis.

🤖 Generated with [Claude Code](https://claude.com/claude-code)

Co-Authored-By: Claude <noreply@anthropic.com>

File: robots/summit_xl_no_arm.urdf.xacro (robot description, xacro)
@@ -25,9 +25,6 @@
 	<xacro:property name="wheel_offset_z" value="0.0" />
 	<xacro:property name="front_laser_offset_x" value="0.356"/>
-	<xacro:property name="front_laser_offset_y" value="-0.251"/>
-	<xacro:property name="front_laser_offset_z" value="0.1566"/>
-    <xacro:property name="rear_laser_offset_x" value="-0.35"/>
-	<xacro:property name="rear_laser_offset_y" value="0.251"/>
-	<xacro:property name="rear_laser_offset_z" value="0.1566"/>
+	<xacro:property name="front_laser_offset_y" value="0.0"/>
+	<xacro:property name="front_laser_offset_z" value="0.25"/>
 	<xacro:property name="front_ptz_camera_offset_x" value="0.308"/>
 	<xacro:property name="front_ptz_camera_offset_y" value="0.141"/>
@@ -78,9 +75,7 @@
 		<!-- SENSORS -->
 		<xacro:sensor_hokuyo_utm30lx_no_frame_prefix ns="$(arg robot_ns)" prefix="front_laser" parent="base_link" min_angle="${-3/4*PI}" max_angle="${3/4*PI}" gpu="false">
-			<origin xyz="${front_laser_offset_x} ${front_laser_offset_y} ${front_laser_offset_z}" rpy="0 0 ${-1/4*PI}" />
+			<origin xyz="${front_laser_offset_x} ${front_laser_offset_y} ${front_laser_offset_z}" rpy="0 0 0" />
   		</xacro:sensor_hokuyo_utm30lx_no_frame_prefix>
-        <xacro:sensor_hokuyo_utm30lx_no_frame_prefix ns="$(arg robot_ns)" prefix="rear_laser" parent="base_link" min_angle="${-3/4*PI}" max_angle="${3/4*PI}" gpu="false">
-			<origin xyz="${rear_laser_offset_x} ${rear_laser_offset_y} ${rear_laser_offset_z}" rpy="0 0 ${3/4*PI}" />
-  		</xacro:sensor_hokuyo_utm30lx_no_frame_prefix>
+		<!-- Rear laser removed - using only front laser -->
 		<!--xacro:sensor_axis_m5013 prefix="$(arg prefix)front_ptz_camera" parent="$(arg prefix)base_link">
 			<origin xyz="${front_ptz_camera_offset_x} ${front_ptz_camera_offset_y} ${front_ptz_camera_offset_z}" rpy="${-PI/2} 0 0"/>
