Commit message: Configure robot to match Yahboom X3 dimensions and meshes
- Updated wheel dimensions to 0.03m radius and width
- Replaced Summit XL meshes with actual Yahboom X3 meshes (base and wheels)
- Adjusted wheel positions (X: 0.08m, Y: 0.085m, Z: -0.039m)
- Raised base height to 0.0815m to match Yahboom configuration
- Repositioned laser to Yahboom location (X: 0.0435m, Z: 0.11m)
- Added Yahboom laser mount mesh (laser_link.STL)
- Reduced laser scan angle from 270° to 240° to avoid self-collision
- Updated IMU position and rotation to match Yahboom specs
- Corrected robot footprint in nav2_params_sim.yaml (0.22m × 0.18m)
- Replaced complex mesh collision with simple box geometry to fix trimesh warnings
- Added mecanum drive plugin with proper wheel parameters

🤖 Generated with [Claude Code](https://claude.com/claude-code)

Co-Authored-By: Claude <noreply@anthropic.com>

File: icclab_summit_xl/icclab_summit_xl/urdf/bases/summit_xl_base.gazebo.xacro (robot description, xacro)
@@ -59,4 +59,17 @@
 		<robot_base_frame>${prefix}base_footprint</robot_base_frame>
       	</plugin>
+		<!-- Mecanum drive to make wheels turn -->
+		<plugin
+        filename="gz-sim-mecanum-drive-system"
+        name="gz::sim::systems::MecanumDrive">
+		<front_left_joint>${prefix}front_left_wheel_joint</front_left_joint>
+		<front_right_joint>${prefix}front_right_wheel_joint</front_right_joint>
+		<back_left_joint>${prefix}rear_left_wheel_joint</back_left_joint>
+		<back_right_joint>${prefix}rear_right_wheel_joint</back_right_joint>
+		<wheel_separation>0.17</wheel_separation>
+		<wheelbase>0.16</wheelbase>
+		<wheel_radius>0.03</wheel_radius>
+		<odom_publish_frequency>50</odom_publish_frequency>
+      	</plugin>
 	  </gazebo>
   </xacro:macro>

File: icclab_summit_xl/icclab_summit_xl/urdf/bases/summit_xl_hls_base.urdf.xacro (robot description, xacro)
@@ -6,6 +6,6 @@
 	  <!-- Robot mechanical and motor parameters -->
 	  <xacro:property name="PI" value="3.1415926535897931"/>
-	  <xacro:property name="wheel_width" value="0.175" />
-    <xacro:property name="wheel_radius" value="0.127" />
+	  <xacro:property name="wheel_width" value="0.03" />
+    <xacro:property name="wheel_radius" value="0.03" />
 	<!-- BASE FOOTPRINT -->
 	  <xacro:if value="${publish_bf}">
@@ -19,5 +19,5 @@
 		</link>
 		<joint name="${prefix}base_footprint_joint" type="fixed">
-		  <origin xyz="0 0 ${wheel_radius}" rpy="0 0 0" /> <!-- ${wheel_radius} property must be defined inside wheel description -->
+		  <origin xyz="0 0 0.0815" rpy="0 0 0" /> <!-- Yahboom base height -->
 		  <parent link="${prefix}base_footprint"/>
 		  <child link="${prefix}base_link" />
@@ -33,14 +33,7 @@
     <visual>
        <origin xyz="0 0 0" rpy="0 0 0" />
-       <xacro:if value="${hq}">
        <geometry>
-	     <mesh filename="file://$(find summit_xl_description)/meshes/bases/hls/summit_xl_hls.stl"/>
+	     <mesh filename="file://$(find icclab_summit_xl)/meshes/mecanum/base_link_X3.STL"/>
        </geometry>
-       </xacro:if>
-       <xacro:unless value="${hq}">
-       <geometry>
-	     <mesh filename="file://$(find summit_xl_description)/meshes/bases/hls/summit_xl_hls.dae"/>
-       </geometry>
-       </xacro:unless>
        <material name="darkgrey">
          <color rgba="0.1 0.1 0.1 1"/>
@@ -50,5 +43,5 @@
        <origin xyz="0 0 0" rpy="0 0 0 " />
        <geometry>
-         <mesh filename="file://$(find summit_xl_description)/meshes/bases/hls/summit_xl_hls.dae"/>
+         <box size="0.200 0.260 0.120"/>
        </geometry>
     </collision>

File: icclab_summit_xl/icclab_summit_xl/urdf/sensors/hokuyo_utm30lx_no_frame_prefix.urdf.xacro (robot description, xacro)
@@ -13,9 +13,13 @@
     </joint>
     <link name="${prefix}_base_link">
+      <!-- Laser mount with sensor -->
       <visual>
-        <origin xyz="0 0 0.055" rpy="0 0 0"/>
+        <origin xyz="0 0 0" rpy="0 0 0"/>
         <geometry>
-            <mesh filename="package://icclab_summit_xl/meshes/hokuyo_utm_30lx.dae"/>
+            <mesh filename="file://$(find icclab_summit_xl)/meshes/sensor/laser_link.STL"/>
         </geometry>
+        <material name="white">
+           <color rgba="1.0 1.0 1.0 1"/>
+        </material>
       </visual>
       <inertial>

File: robots/summit_xl_no_arm.urdf.xacro (robot description, xacro)
@@ -9,5 +9,5 @@
 	<xacro:include filename="$(find icclab_summit_xl)/urdf/bases/summit_xl_hls_base.urdf.xacro" />
 	<!-- Import summit XL wheels -->
-	<xacro:include filename="$(find summit_xl_description)/urdf/wheels/omni_wheel.urdf.xacro" />
+	<xacro:include filename="$(find icclab_summit_xl)/urdf/wheels/omni_wheel.urdf.xacro" />
 	<xacro:include filename="$(find summit_xl_description)/urdf/wheels/rubber_wheel.urdf.xacro" />
 	<xacro:include filename="$(find summit_xl_description)/urdf/structures/structure_hokuyo.urdf.xacro" />
@@ -17,26 +17,18 @@
 	<xacro:include filename="$(find icclab_summit_xl)/urdf/sensors/intel_camera_mount.urdf.xacro" />
 	<xacro:include filename="$(find icclab_summit_xl)/urdf/sensors/imu_hector_plugin.urdf.xacro"/>
-	<!-- Arm and gripper removed for no-arm configuration -->
 	<xacro:property name="PI" value="3.1415926535897931"/>
 	<!-- Wheel parameters -->
-	<!-- Wheel parameters -->
-	<xacro:property name="wheel_offset_x" value="0.2225" />    <!-- x,y,z in translation from base_link to the center of the wheel -->
-	<xacro:property name="wheel_offset_y" value="0.2045" />
-	<xacro:property name="wheel_offset_z" value="0.0" />
-	<xacro:property name="front_laser_offset_x" value="0.356"/>
+	<xacro:property name="wheel_offset_x" value="0.08" />    <!-- x,y,z in translation from base_link to the center of the wheel -->
+	<xacro:property name="wheel_offset_y" value="0.085" />
+	<xacro:property name="wheel_offset_z" value="-0.039" /> <!-- Yahboom wheel height -->
+	<xacro:property name="front_laser_offset_x" value="0.0435"/>
 	<xacro:property name="front_laser_offset_y" value="0.0"/>
-	<xacro:property name="front_laser_offset_z" value="0.25"/>
-	<xacro:property name="front_ptz_camera_offset_x" value="0.308"/>
-	<xacro:property name="front_ptz_camera_offset_y" value="0.141"/>
-	<xacro:property name="front_ptz_camera_offset_z" value="0.195"/>
-	<xacro:property name="rear_ptz_camera_offset_x" value="-0.308"/>
-	<xacro:property name="rear_ptz_camera_offset_y" value="-0.141"/>
-	<xacro:property name="rear_ptz_camera_offset_z" value="0.195"/>
-	<xacro:property name="imu_offset_x" value="0.127"/>
-	<xacro:property name="imu_offset_y" value="-0.129"/>
-	<xacro:property name="imu_offset_z" value="0.212"/>
-	<xacro:property name="front_rgbd_camera_offset_x" value="0.35850"/>
+	<xacro:property name="front_laser_offset_z" value="0.11"/>
+	<xacro:property name="imu_offset_x" value="-0.06"/>
+	<xacro:property name="imu_offset_y" value="0.025"/>
+	<xacro:property name="imu_offset_z" value="0.095"/>
+	<xacro:property name="front_rgbd_camera_offset_x" value="0.087"/>
 	<xacro:property name="front_rgbd_camera_offset_y" value="0.0"/>
-	<xacro:property name="front_rgbd_camera_offset_z" value="0.22062"/>
+	<xacro:property name="front_rgbd_camera_offset_z" value="0.037"/>
 	<xacro:property name="gps_offset_x" value="-0.365"/>
 	<xacro:property name="gps_offset_y" value="-0.167"/>
@@ -71,17 +63,10 @@
         <!-- IMU -->
 		<xacro:sensor_imu_hector prefix="$(arg prefix)imu" ns="$(arg robot_ns)" parent="$(arg prefix)base_link">
-			<origin xyz="${imu_offset_x} ${imu_offset_y} ${imu_offset_z}" rpy="0 0 0"/>
+			<origin xyz="${imu_offset_x} ${imu_offset_y} ${imu_offset_z}" rpy="0 ${PI} ${PI/2}"/>
 		</xacro:sensor_imu_hector>
 		<!-- SENSORS -->
-		<xacro:sensor_hokuyo_utm30lx_no_frame_prefix ns="$(arg robot_ns)" prefix="front_laser" parent="base_link" min_angle="${-3/4*PI}" max_angle="${3/4*PI}" gpu="false">
+		<xacro:sensor_hokuyo_utm30lx_no_frame_prefix ns="$(arg robot_ns)" prefix="front_laser" parent="base_link" min_angle="${-12*PI/18}" max_angle="${12*PI/18}" gpu="false">
 			<origin xyz="${front_laser_offset_x} ${front_laser_offset_y} ${front_laser_offset_z}" rpy="0 0 0" />
   		</xacro:sensor_hokuyo_utm30lx_no_frame_prefix>
-		<!-- Rear laser removed - using only front laser -->
-		<!--xacro:sensor_axis_m5013 prefix="$(arg prefix)front_ptz_camera" parent="$(arg prefix)base_link">
-			<origin xyz="${front_ptz_camera_offset_x} ${front_ptz_camera_offset_y} ${front_ptz_camera_offset_z}" rpy="${-PI/2} 0 0"/>
-		</xacro:sensor_axis_m5013-->
-		<!--xacro:sensor_axis_m5013 prefix="$(arg prefix)rear_ptz_camera" parent="$(arg prefix)base_link">
-			<origin xyz="${rear_ptz_camera_offset_x} ${rear_ptz_camera_offset_y} ${rear_ptz_camera_offset_z}" rpy="${-PI/2} 0 ${PI}"/>
-		</xacro:sensor_axis_m5013-->
 		<xacro:sensor_d435_icclab prefix="$(arg prefix)front_rgbd_camera" parent="$(arg prefix)base_link" ns="$(arg robot_ns)">
 			<origin xyz="${front_rgbd_camera_offset_x} ${front_rgbd_camera_offset_y} ${front_rgbd_camera_offset_z}" rpy="0 0 0"/>
@@ -90,5 +75,4 @@
 			<origin xyz="${gps_offset_x} ${gps_offset_y} ${gps_offset_z}" rpy="0 0 0"/>
 		</xacro:sensor_gps-->
-		<!-- Arm, gripper, and Luxonis camera removed -->
    </xacro:macro>
    <xacro:summit_xl prefix="$(arg prefix)" publish_bf="true" hq="true"/>
