Commit message: Working gazebo config: /tmp/.X11-unix/gazebo.config

File: icclab_summit_xl/icclab_summit_xl/urdf/sensors/imu_hector_plugin.urdf.xacro (robot description, xacro)
@@ -1,4 +1,10 @@
 <?xml version="1.0"?>
 <robot name="sensor_imu" xmlns:xacro="http://wiki.ros.org/xacro">
+  <!-- Inertia macro for a solid cuboid (box) -->
+  <xacro:macro name="solid_cuboid_inertia" params="m w h d">
+    <inertia ixx="${m*(h*h+d*d)/12}" ixy="0" ixz="0"
+             iyy="${m*(w*w+d*d)/12}" iyz="0"
+             izz="${m*(w*w+h*h)/12}" />
+  </xacro:macro>
   <xacro:macro name="sensor_imu_hector" params="ns prefix topic:='imu/data' parent *origin">
     <joint name="${prefix}_joint" type="fixed">

File: robots/summit_xl_no_arm.urdf.xacro (robot description, xacro)
@@ -10,10 +10,7 @@
 	<!-- Import summit XL wheels -->
 	<xacro:include filename="$(find icclab_summit_xl)/urdf/wheels/omni_wheel.urdf.xacro" />
-	<xacro:include filename="$(find summit_xl_description)/urdf/wheels/rubber_wheel.urdf.xacro" />
-	<xacro:include filename="$(find summit_xl_description)/urdf/structures/structure_hokuyo.urdf.xacro" />
-	<!-- Import our modified sensor -->
+	<!-- Import sensors -->
 	<xacro:include filename="$(find icclab_summit_xl)/urdf/sensors/hokuyo_utm30lx_no_frame_prefix.urdf.xacro" />
 	<xacro:include filename="$(find icclab_summit_xl)/urdf/sensors/intel_d435.urdf.xacro" />
-	<xacro:include filename="$(find icclab_summit_xl)/urdf/sensors/intel_camera_mount.urdf.xacro" />
 	<xacro:include filename="$(find icclab_summit_xl)/urdf/sensors/imu_hector_plugin.urdf.xacro"/>
 	<xacro:property name="PI" value="3.1415926535897931"/>
